Commit message: added pressure subscriber to gazebo_hardware_node, moved depth sensor to center of mass in qubo.xacro file

File: src/qubo_gazebo/urdf/basic_qubo.xacro (robot description, xacro)
@@ -184,5 +184,5 @@
   <!-- Pressure  -->
   <xacro:default_pressure namespace="${namespace}" parent_link="${namespace}/base_link">
-    <origin xyz="-1.32 0.5 0.85" rpy="0 0 0"/>
+    <origin xyz="0 0 0" rpy="0 0 0"/>
   </xacro:default_pressure>
   <!-- IMU  -->

Commit message: modified qubo.xacro file so the weight is more in line with actual qubo, also changed the comment style so that emacs doesn't choke when I try to comment stuff, modified depth controller to actually read in the current depth

File: src/qubo_gazebo/urdf/basic_qubo.xacro (robot description, xacro)
@@ -9,5 +9,5 @@
   <xacro:property name="prop_mesh_file" value="file://$(find uuv_descriptions)/models/rexrov/mesh/prop.dae"/>
   <!-- Qubo's mass, volume, and center of buoyancy -->
-  <xacro:property name="mass" value="1862.87"/>
+  <xacro:property name="mass" value="18.6287"/>
   <xacro:property name="volume" value="1.83826"/>
   <xacro:property name="center_of_buoyancy" value="0.0 0.0 0.3"/>
@@ -49,5 +49,5 @@
         <conversion>
           <type>Basic</type>
-          <rotorConstant>0.00031</rotorConstant>
+          <rotorConstant>-1</rotorConstant>
         </conversion>
       </plugin>
@@ -83,8 +83,8 @@
     <limit effort="0" lower="0" upper="0" velocity="0"/>
   </joint>
-  <!-- Set up hydrodynamic plugin -->
+  <!-- Set up hydrodynamic plugin  -->
   <gazebo>
     <plugin name="uuv_plugin" filename="libunderwater_object_ros_plugin.so">
-      <fluid_density>1028.0</fluid_density>
+      <fluid_density>10.280</fluid_density>
       <flow_velocity_topic>hydrodynamics/current_velocity</flow_velocity_topic>
       <debug>${debug}</debug>
@@ -93,24 +93,24 @@
         <volume>${volume}</volume>
         <box>
-          <width>1.0</width>
-          <length>1.0</length>
-          <height>1.0</height>
+          <width>.4064</width>
+          <length>.3048</length>
+          <height>.3048</height>
         </box>
         <center_of_buoyancy>${center_of_buoyancy}</center_of_buoyancy>
-        <!-- Added mass: see p.28 in Berg2012 -->
+  <!-- Added mass: see p.28 in Berg2012 -->
         <hydrodynamic_model>
           <type>fossen</type>
           <added_mass>
-             779.79 -6.8773 -103.32 8.5426 -165.54 -7.8033
-            -6.8773 1222 51.29 409.44 -5.8488 62.726
-              -103.32 51.29 3659.9 6.1112 -386.42 10.774
-              8.5426 409.44 6.1112 534.9 -10.027 21.019
-              -165.54 -5.8488 -386.42 -10.027 842.69 -1.1162
-              -7.8033 62.726 10.775 21.019 -1.1162 224.32
+             7.7979 -0.068773 -1.0332 .085426 -1.6554 -.078033
+            -.068773 12.22 0.5129 4.0944 -0.058488 0.62726
+              -1.0332 0.5129 36.599 0.61112 -3.8642 0.10774
+              .085426 4.0944 .061112 5.349 -0.10027 0.21019
+              -1.6554 -.058488 -3.8642 -0.10027 8.4269 -.011162
+              -.078033 0.62726 0.10775 0.21019 -.011162 2.2432
           </added_mass>
-          <!-- Linear damping: see p.31 in Berg2012 -->
-          <linear_damping>-74.82 -69.48 -728.4 -268.8 -309.77 -105</linear_damping>
+           <!-- Linear damping: see p.31 in Berg2012 -->
+          <linear_damping>-0.7482 -0.6948 -7.284 -2.688 -3.0977 -105</linear_damping>
           <!-- Non-linear damping: see p.30 in Berg2012 -->
-          <quadratic_damping>-748.22 -992.53 -1821.01 -672 -774.44 -523.27</quadratic_damping>
+          <quadratic_damping>-7.4822 -9.9253 -18.2101 -6.72 -7.7444 -5.2327</quadratic_damping>
         </hydrodynamic_model>
       </link>
@@ -195,4 +195,4 @@
   </xacro:default_camera>
   <!-- Joint state publisher -->
-  <xacro:default_joint_state_publisher namespace="qubo_test" update_rate="500"/>
+<!--  <xacro:default_joint_state_publisher namespace="qubo_test" update_rate="500"/> -->
 </robot>

Commit message: [Made vehicle simulation parameters more realistic, not sure if correct yet]

File: src/qubo_gazebo/urdf/basic_qubo.xacro (robot description, xacro)
@@ -10,6 +10,6 @@
   <!-- Qubo's mass, volume, and center of buoyancy -->
   <xacro:property name="mass" value="18.6287"/>
-  <xacro:property name="volume" value="1.83826"/>
-  <xacro:property name="center_of_buoyancy" value="0.0 0.0 0.3"/>
+  <xacro:property name="volume" value="0.037"/>
+  <xacro:property name="center_of_buoyancy" value="-0.02 0.0 0.16"/>
   <!-- Thruster joint and link macro -->
   <xacro:macro name="thruster_macro" params="namespace thruster_id *origin">
@@ -86,5 +86,5 @@
   <gazebo>
     <plugin name="uuv_plugin" filename="libunderwater_object_ros_plugin.so">
-      <fluid_density>10.280</fluid_density>
+      <fluid_density>1000.0</fluid_density>
       <flow_velocity_topic>hydrodynamics/current_velocity</flow_velocity_topic>
       <debug>${debug}</debug>
@@ -178,8 +178,4 @@
     </plugin>
   </gazebo>
-  <!-- DVL -->
-  <xacro:default_dvl namespace="${namespace}" parent_link="${namespace}/base_link">
-    <origin xyz="-1.4 0 -0.312" rpy="0 ${0.5*pi} 0"/>
-  </xacro:default_dvl>
   <!-- Pressure  -->
   <xacro:default_pressure namespace="${namespace}" parent_link="${namespace}/base_link">
@@ -192,5 +188,5 @@
   <!-- Camera -->
   <xacro:default_camera namespace="${namespace}" parent_link="${namespace}/base_link">
-    <origin xyz="1.15 0 0.4" rpy="0 0.6 0"/>
+    <origin xyz="0.25 0 0" rpy="0 1.57 0"/>
   </xacro:default_camera>
   <!-- Joint state publisher -->
