Commit message: updated basic_qubo.xacro so the camera is in the right spot

File: src/vl_qubo_gazebo/urdf/basic_qubo.xacro (robot description, xacro)
@@ -179,7 +179,7 @@
   </gazebo>
   <!-- DVL -->
-  <xacro:default_dvl namespace="${namespace}" parent_link="${namespace}/base_link">
-    <origin xyz="-1.4 0 -0.312" rpy="0 ${0.5*pi} 0"/>
-  </xacro:default_dvl>
+  <!-- <xacro:default_dvl namespace="${namespace}" parent_link="${namespace}/base_link"> -->
+  <!--   <origin xyz="-1.4 0 -0.312" rpy="0 ${0.5*pi} 0"/> -->
+  <!-- </xacro:default_dvl> -->
   <!-- Pressure  -->
   <xacro:default_pressure namespace="${namespace}" parent_link="${namespace}/base_link">
@@ -192,5 +192,5 @@
   <!-- Camera -->
   <xacro:default_camera namespace="${namespace}" parent_link="${namespace}/base_link">
-    <origin xyz="1.15 0 0.4" rpy="0 0.6 0"/>
+    <origin xyz=".35 0 0.15" rpy="0 0 0"/>
   </xacro:default_camera>
   <!-- Joint state publisher -->

File: src/vl_qubo_gazebo/urdf/mesh_qubo.xacro (robot description, xacro)
@@ -8,5 +8,5 @@
   <xacro:property name="namespace" value="basic_qubo"/>
   <xacro:property name="prop_mesh_file" value="file://$(find uuv_descriptions)/models/rexrov/mesh/prop.dae"/>
-  <xacro:property name="frame_mesh_file" value="file://$(find uuv_descriptions)/models/rexrov/mesh/prop.dae"/>
+  <xacro:property name="frame_mesh_file" value="file://prop.dae"/>
   <!-- Qubo's mass, volume, and center of buoyancy -->
   <xacro:property name="mass" value="18.6287"/>
@@ -181,7 +181,7 @@
   </gazebo>
   <!-- DVL -->
-  <xacro:default_dvl namespace="${namespace}" parent_link="${namespace}/base_link">
-    <origin xyz="-1.4 0 -0.312" rpy="0 ${0.5*pi} 0"/>
-  </xacro:default_dvl>
+  <!-- <xacro:default_dvl namespace="${namespace}" parent_link="${namespace}/base_link"> -->
+  <!--   <origin xyz="-1.4 0 -0.312" rpy="0 ${0.5*pi} 0"/> -->
+  <!-- </xacro:default_dvl> -->
   <!-- Pressure  -->
   <xacro:default_pressure namespace="${namespace}" parent_link="${namespace}/base_link">

Commit message: [Updated moments of inertia]

File: src/vl_qubo_gazebo/urdf/basic_qubo.xacro (robot description, xacro)
@@ -71,5 +71,5 @@
       <mass value="${mass}"/>
       <origin xyz="0 0 0"/>
-      <inertia ixx="525.39" ixy="1.44" ixz="33.41" iyy="794.20" iyz="2.6" izz="691.23"/>
+      <inertia ixx="0.297155" ixy="-0.0026542" ixz="0.0079437" iyy="0.435426" iyz="0.003223" izz="0.570213"/>
     </inertial>
   </link>

Commit message: added some debug stuff

File: src/vl_qubo_gazebo/urdf/basic_qubo.xacro (robot description, xacro)
@@ -9,6 +9,6 @@
   <xacro:property name="prop_mesh_file" value="file://$(find uuv_descriptions)/models/rexrov/mesh/prop.dae"/>
   <!-- Qubo's mass, volume, and center of buoyancy -->
-  <xacro:property name="mass" value="18.6287"/>
-  <xacro:property name="volume" value="0.037"/>
+  <xacro:property name="mass" value="15.87"/>
+  <xacro:property name="volume" value=".018"/>
   <xacro:property name="center_of_buoyancy" value="0.0 0.0 0.16"/>
   <!-- Thruster joint and link macro -->
@@ -90,5 +90,5 @@
       <debug>${debug}</debug>
       <link name="${namespace}/base_link">
-        <neutrally_buoyant>0</neutrally_buoyant>
+        <neutrally_buoyant>1</neutrally_buoyant>
         <volume>${volume}</volume>
         <box>
@@ -144,8 +144,8 @@
   </xacro:thruster_macro>
   <xacro:thruster_macro namespace="${namespace}" thruster_id="6">
-    <origin xyz="0.149 0.083 0" rpy="${0*d2r} ${-90*d2r} ${0*d2r}"/>
+    <origin xyz="0.257 0.083 0" rpy="${0*d2r} ${-90*d2r} ${0*d2r}"/>
   </xacro:thruster_macro>
   <xacro:thruster_macro namespace="${namespace}" thruster_id="7">
-    <origin xyz="0.149 -0.083 0" rpy="${0*d2r} ${-90*d2r} ${0*d2r}"/>
+    <origin xyz="0.257 -0.083 0" rpy="${0*d2r} ${-90*d2r} ${0*d2r}"/>
   </xacro:thruster_macro>
   <!-- Mount a 3D pose sensor -->

Commit message: updating .xacro file again

File: src/vl_qubo_gazebo/urdf/basic_qubo.xacro (robot description, xacro)
@@ -71,5 +71,5 @@
       <mass value="${mass}"/>
       <origin xyz="0 0 0"/>
-      <inertia ixx="0.297155" ixy="-0.0026542" ixz="0.0079437" iyy="0.435426" iyz="0.003223" izz="0.570213"/>
+      <inertia ixx="0.297155" ixy="0.0026542" ixz="0.0079437" iyy="0.435426" iyz="0.003223" izz="0.570213"/>
     </inertial>
   </link>

Commit message: changed up our depth sensor, played around with ROS pid but will probably movve back to our own, also removed the tf node in spawn_basic qubo

File: src/vl_qubo_gazebo/urdf/basic_qubo.xacro (robot description, xacro)
@@ -169,4 +169,23 @@
     <limit effort="0" lower="0" upper="0" velocity="0"/>
   </joint>
+  <!-- Mount a 3D pose sensor -->
+  <link name="${namespace}/pressure_link">
+    <xacro:box_inertial x="0" y="0" z="0" mass="0.01">
+      <origin xyz="0 0 0" rpy="0 0 0"/>
+    </xacro:box_inertial>
+    <visual>
+      <geometry>
+        <box size="0.1 0.1 0.1"/>
+      </geometry>
+    </visual>
+    <xacro:no_collision/>
+  </link>
+  <joint name="${namespace}/pressure_joint" type="revolute">
+    <origin xyz="0 0 0" rpy="0 0 0"/>
+    <axis xyz="0 0 1"/>
+    <parent link="${namespace}/base_link"/>
+    <child link="${namespace}/pressure_link"/>
+    <limit effort="0" lower="0" upper="0" velocity="0"/>
+  </joint>
   <gazebo>
     <plugin name="pose_3d_plugin" filename="libgazebo_ros_p3d.so">
@@ -178,4 +197,15 @@
       <updateRate>30</updateRate>
     </plugin>
+    <plugin filename="libuuv_gazebo_ros_subseapressure.so" name="libuuv_gazebo_subseapressure_plugin">
+      <robotNamespace>${namespace}</robotNamespace> <!-- (string, required): ros namespace in which the messages are published -->
+      <linkName>${namespace}/pressure_link</linkName> <!-- (string, required): name of the body which holds the IMU sensor -->
+      <sensorTopic>pressure</sensorTopic>
+      <updatePeriod>.016</updatePeriod> <!-- Update period of accelerometer and gyroscope [s] -->
+      <range>3000</range> <!-- measurement range [kPa] -->
+      <stddev>1.66</stddev> <!-- measurement stddev [kPa] -->
+      <estimateDepth>false</estimateDepth> <!-- infer depth? -->
+      <standardPressure>101.325</standardPressure> <!-- pressure at sea level (depth 0 m) [kPa] -->
+      <kPaPerM>9.803</kPaPerM> <!-- increase in pressure [kPa] per [m] in increased depth -->
+  </plugin>
   </gazebo>
   <!-- DVL -->
@@ -184,7 +214,9 @@
   <!-- </xacro:default_dvl> -->
   <!-- Pressure  -->
-  <xacro:default_pressure namespace="${namespace}" parent_link="${namespace}/base_link">
-    <origin xyz="0 0 0" rpy="0 0 0"/>
-  </xacro:default_pressure>
+  <!-- <xacro:default_pressure namespace="${namespace}" parent_link="${namespace}/base_link"> -->
+  <!--   <origin xyz="0 0 0" rpy="0 0 0"/> -->
+  <!--   <stddev>.01</stddev> -->
+  <!-- </xacro:default_pressure> -->
+  <!-- these should match the bar 30 on qubo, up to 300 kpa , with an absolute error absolute error of 5 kpa I assumed absolute error is about 3 * stddevs giving std dev of   -->
   <!-- IMU  -->
   <xacro:default_imu namespace="${namespace}" parent_link="${namespace}/base_link">

Commit message: cleaned up a little, no functional changes

File: src/vl_qubo_gazebo/urdf/basic_qubo.xacro (robot description, xacro)
@@ -12,46 +12,4 @@
   <xacro:property name="volume" value=".018"/>
   <xacro:property name="center_of_buoyancy" value="0.0 0.0 0.16"/>
-  <!-- Thruster joint and link macro -->
-  <xacro:macro name="thruster_macro" params="namespace thruster_id *origin">
-    <joint name="${namespace}/thruster_${thruster_id}_joint" type="continuous">
-      <xacro:insert_block name="origin"/>
-      <axis xyz="1 0 0"/>
-      <parent link="${namespace}/base_link"/>
-      <child link="${namespace}/thruster_${thruster_id}"/>
-    </joint>
-    <link name="${namespace}/thruster_${thruster_id}">
-      <xacro:box_inertial x="0" y="0" z="0" mass="0.001">
-        <origin xyz="0 0 0" rpy="0 0 0"/>
-      </xacro:box_inertial>
-      <visual>
-        <origin rpy="0 0 0" xyz="0 0 0"/>
-        <geometry>
-          <mesh filename="${prop_mesh_file}" scale=".5 .5 .5"/>
-        </geometry>
-      </visual>
-      <collision>
-        <origin xyz="0 0 0" rpy="0 ${0.5*pi} 0"/>
-        <geometry>
-          <cylinder length="0.000001" radius="0.000001"/>
-        </geometry>
-      </collision>
-    </link>
-    <gazebo>
-      <plugin name="${namespace}_${thruster_id}_thruster_model" filename="libthruster_ros_plugin.so">
-        <linkName>${namespace}/thruster_${thruster_id}</linkName>
-        <jointName>${namespace}/thruster_${thruster_id}_joint</jointName>
-        <thrustTopic>${namespace}/thrusters/${thruster_id}/thrust</thrustTopic>
-        <inputTopic>${namespace}/thrusters/${thruster_id}/input</inputTopic>
-        <dynamics>
-          <type>FirstOrder</type>
-          <timeConstant>0.05</timeConstant>
-        </dynamics>
-        <conversion>
-          <type>Basic</type>
-          <rotorConstant>-.05</rotorConstant>
-        </conversion>
-      </plugin>
-    </gazebo>
-  </xacro:macro>
   <!-- size of robot to meters X = .4064Z  Y = Z = .3048 -->
   <!-- Qubo's base link. Assume a right-handed coordinate system, with x forward and z up -->
@@ -118,4 +76,48 @@
     </plugin>
   </gazebo>
+  <!-- thrusters -->
+  <!-- ============================================================================== -->
+    <!-- Thruster joint and link macro -->
+  <xacro:macro name="thruster_macro" params="namespace thruster_id *origin">
+    <joint name="${namespace}/thruster_${thruster_id}_joint" type="continuous">
+      <xacro:insert_block name="origin"/>
+      <axis xyz="1 0 0"/>
+      <parent link="${namespace}/base_link"/>
+      <child link="${namespace}/thruster_${thruster_id}"/>
+    </joint>
+    <link name="${namespace}/thruster_${thruster_id}">
+      <xacro:box_inertial x="0" y="0" z="0" mass="0.001">
+        <origin xyz="0 0 0" rpy="0 0 0"/>
+      </xacro:box_inertial>
+      <visual>
+        <origin rpy="0 0 0" xyz="0 0 0"/>
+        <geometry>
+          <mesh filename="${prop_mesh_file}" scale=".5 .5 .5"/>
+        </geometry>
+      </visual>
+      <collision>
+        <origin xyz="0 0 0" rpy="0 ${0.5*pi} 0"/>
+        <geometry>
+          <cylinder length="0.000001" radius="0.000001"/>
+        </geometry>
+      </collision>
+    </link>
+    <gazebo>
+      <plugin name="${namespace}_${thruster_id}_thruster_model" filename="libthruster_ros_plugin.so">
+        <linkName>${namespace}/thruster_${thruster_id}</linkName>
+        <jointName>${namespace}/thruster_${thruster_id}_joint</jointName>
+        <thrustTopic>${namespace}/thrusters/${thruster_id}/thrust</thrustTopic>
+        <inputTopic>${namespace}/thrusters/${thruster_id}/input</inputTopic>
+        <dynamics>
+          <type>FirstOrder</type>
+          <timeConstant>0.05</timeConstant>
+        </dynamics>
+        <conversion>
+          <type>Basic</type>
+          <rotorConstant>-.05</rotorConstant>
+        </conversion>
+      </plugin>
+    </gazebo>
+  </xacro:macro>
   <!-- yaw thrusters - Z = 5 inches from bottom, X = 9.28 inches from center, Y = 7.87 inches from center -->
   <!-- Z = .127 X = .23 Y = .1998 -->
@@ -150,4 +152,6 @@
     <origin xyz="0.257 -0.083 0" rpy="${0*d2r} ${-90*d2r} ${0*d2r}"/>
   </xacro:thruster_macro>
+  <!-- sensors -->
+  <!-- ============================================================================== -->
   <!-- Mount a 3D pose sensor -->
   <link name="${namespace}/pose_sensor_link">

Commit message: cleaned up our simulators namsepacesaccounted for that in the controller as well

File: src/vl_qubo_gazebo/urdf/basic_qubo.xacro (robot description, xacro)
@@ -1,4 +1,4 @@
 <?xml version="1.0"?>
-<robot name="qubo_test" xmlns:xacro="http://www.ros.org/wiki/xacro" >
+<robot name="gazebo_qubo" xmlns:xacro="http://www.ros.org/wiki/xacro" >
   <!-- Includes -->
   <xacro:include filename="$(find uuv_descriptions)/models/common/urdf/common.urdf.xacro"/>
@@ -6,5 +6,6 @@
   <!-- Parameters -->
   <xacro:property name="debug" value="0"/>
-  <xacro:property name="namespace" value="basic_qubo"/>
+  <!-- don't be fooled, if you want to change qubo's namespace, change the parameter below , and the name parameter above -->
+  <xacro:property name="namespace" value="gazebo_qubo"/>
   <xacro:property name="prop_mesh_file" value="file://$(find uuv_descriptions)/models/rexrov/mesh/prop.dae"/>
   <!-- Qubo's mass, volume, and center of buoyancy -->
@@ -78,5 +79,5 @@
   <!-- thrusters -->
   <!-- ============================================================================== -->
-    <!-- Thruster joint and link macro -->
+  <!-- Thruster joint and link macro -->
   <xacro:macro name="thruster_macro" params="namespace thruster_id *origin">
     <joint name="${namespace}/thruster_${thruster_id}_joint" type="continuous">
@@ -229,5 +230,6 @@
   </xacro:default_imu>
   <!-- Camera -->
-  <xacro:default_camera namespace="${namespace}" parent_link="${namespace}/base_link">
+  <!-- the camera used the robot name + given namespace as it's namespace, so we omit the latter since the robot name is our namespace -->
+  <xacro:default_camera namespace="" parent_link="${namespace}/base_link">
     <origin xyz=".35 0 0.15" rpy="0 0 0"/>
   </xacro:default_camera>

Commit message: changed our hydrodynamic plugin to have positive bouyancy (rather than perfectly nuetral

File: src/vl_qubo_gazebo/urdf/basic_qubo.xacro (robot description, xacro)
@@ -11,5 +11,5 @@
   <!-- Qubo's mass, volume, and center of buoyancy -->
   <xacro:property name="mass" value="15.87"/>
-  <xacro:property name="volume" value=".018"/>
+  <xacro:property name="volume" value=".0165"/>
   <xacro:property name="center_of_buoyancy" value="0.0 0.0 0.16"/>
   <!-- size of robot to meters X = .4064Z  Y = Z = .3048 -->
@@ -49,5 +49,5 @@
       <debug>${debug}</debug>
       <link name="${namespace}/base_link">
-        <neutrally_buoyant>1</neutrally_buoyant>
+        <neutrally_buoyant>0</neutrally_buoyant>
         <volume>${volume}</volume>
         <box>
@@ -88,5 +88,5 @@
     </joint>
     <link name="${namespace}/thruster_${thruster_id}">
-      <xacro:box_inertial x="0" y="0" z="0" mass="0.001">
+      <xacro:box_inertial x="0" y="0" z="0" mass="0.01">
         <origin xyz="0 0 0" rpy="0 0 0"/>
       </xacro:box_inertial>
@@ -200,5 +200,5 @@
       <topicName>pose_gt</topicName>
       <frameName>world</frameName>
-      <gaussianNoise>0.0</gaussianNoise>
+      <gaussianNoise>0.0349</gaussianNoise> <!-- our noise from the AHRS is 2 degrees rms -->
       <updateRate>30</updateRate>
     </plugin>
